File: keeb-kicad/keeb-kicad.kicad_pcb (KiCad board)
At the start: 2 copper layers, 315 x 135 mm, 147 parts, among them SW1 SW_Push, SW10 SW_Push, SW11 SW_Push, SW12 SW_Push, SW13 SW_Push, SW14 SW_Push, SW15 SW_Push, SW16 SW_Push, SW17 SW_Push, SW18 SW_Push, SW19 SW_Push, SW2 SW_Push, SW20 SW_Push, SW21 SW_Push, SW22 SW_Push, SW23 SW_Push, SW24 SW_Push, SW25 SW_Push, SW26 SW_Push, SW27 SW_Push, SW28 SW_Push, SW29 SW_Push, SW3 SW_Push, SW30 SW_Push, SW31 SW_Push, SW32 SW_Push, SW33 SW_Push, SW34 SW_Push, SW35 SW_Push, SW36 SW_Push, SW37 SW_Push, SW38 SW_Push, SW39 SW_Push, SW4 SW_Push, SW40 SW_Push, SW41 SW_Push, SW42 SW_Push, SW43 SW_Push, SW44 SW_Push, SW45 SW_Push, SW46 SW_Push, SW47 SW_Push, SW48 SW_Push, SW49 SW_Push, SW5 SW_Push, SW50 SW_Push, SW51 SW_Push, SW52 SW_Push, SW53 SW_Push, SW54 SW_Push, SW55 SW_Push, SW56 SW_Push, SW57 SW_Push, SW58 SW_Push, SW59 SW_Push, SW6 SW_Push, SW60 SW_Push, SW61 SW_Push, SW62 SW_Push, SW63 SW_Push, SW64 SW_Push, SW65 SW_Push, SW66 SW_Push, SW67 SW_Push, SW68 SW_Push, SW69 SW_Push, SW7 SW_Push, SW70 SW_Push, SW71 RotaryEncoder_Switch, SW8 SW_Push, SW9 SW_Push

Commit message: Placed rest of the components onto PCB
Parts:
- moved SW71 360.7 mm to (0.79, 31.9)
- moved D60 357.4 mm to (3.52, 138.0), turned to 90 degrees
- moved D61 338.2 mm to (22.6, 138.0), turned to 90 degrees
- moved D46 326.5 mm to (22.6, 119.0), turned to 90 degrees
- moved D32 320.4 mm to (17.8, 99.9), turned to 90 degrees
- moved D62 318.9 mm to (41.6, 138.0), turned to 90 degrees
- moved D1 315.1 mm to (3.54, 61.8), turned to 90 degrees
- moved D16 314.8 mm to (13.2, 80.9), turned to 90 degrees
- moved D47 307.4 mm to (41.6, 119.0), turned to 90 degrees
- moved D33 301.5 mm to (36.9, 99.9), turned to 90 degrees
- moved D63 299.7 mm to (60.7, 138.0), turned to 90 degrees
- moved D48 299.4 mm to (60.7, 119.0), turned to 90 degrees
- moved D2 296.6 mm to (22.6, 61.8), turned to 90 degrees
- moved D17 296.0 mm to (32.3, 80.9), turned to 90 degrees
- moved D34 282.6 mm to (55.9, 99.9), turned to 90 degrees
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- renumbered D59 to D48, D48 to D49, D49 to D50, D50 to D51, D51 to D52, D52 to D53, D53 to D54, D54 to D55, D55 to D56, D56 to D57, D57 to D58, D58 to D59
Other:
- board size 315 x 135 mm -> 329 x 135 mm

Commit message: Finished route tracing and added ground fill
Parts:
- moved A1 4.11 mm to (308.1, 28.5)
- moved D44 0.74 mm to (284.5, 99.9)
Connections:
- A1 pad 1: /ROW0 -> /COL0
- A1 pad 10: /COL2 -> /COL7
- A1 pad 11: /COL3 -> /COL8
- A1 pad 12: /COL4 -> /COL9
- A1 pad 14: /COL5 -> /COL10
- A1 pad 15: /COL6 -> /COL11
- A1 pad 16: /COL7 -> /COL12
- A1 pad 17: /COL8 -> /COL13
- A1 pad 19: /COL9 -> /COL14
- A1 pad 2: /ROW1 -> /COL1
- A1 pad 20: /COL10 -> /COL15
- A1 pad 21: /COL11 -> /SWITCH1
- A1 pad 22: /COL12 -> /ENC_B
- A1 pad 24: /COL13 -> /ENC_A
- A1 pad 25: /COL14 -> /ROW0
- A1 pad 26: /COL15 -> /ROW1
- A1 pad 27: /ENC_A -> /ROW2
- A1 pad 29: /ENC_B -> /ROW3
- A1 pad 31: /SWITCH1 -> /ROW4
- A1 pad 4: /ROW2 -> /COL2
- A1 pad 5: /ROW3 -> /COL3
- A1 pad 6: /ROW4 -> /COL4
- A1 pad 7: /COL0 -> /COL5
- A1 pad 9: /COL1 -> /COL6
- D48 pad 1: unconnected-(D48-K-Pad1) -> /ROW3
Routing:
- net /COL0: track 0.00 -> 440.7 mm
- net /ROW4: track 0.00 -> 412.3 mm
- net /COL1: track 0.00 -> 409.6 mm
- net /COL2: track 0.00 -> 385.1 mm
- net /ROW3: track 0.00 -> 378.4 mm
- net /ROW2: track 0.00 -> 368.4 mm
- net /COL3: track 0.00 -> 364.3 mm
- net /ROW1: track 0.00 -> 355.8 mm
- net /ROW0: track 0.00 -> 350.1 mm
- net /COL4: track 0.00 -> 311.5 mm
- net /ENC_A: track 0.00 -> 292.9 mm
- net /COL5: track 0.00 -> 290.2 mm
- net /COL6: track 0.00 -> 287.1 mm
- net /ENC_B: track 0.00 -> 279.5 mm
- net /SWITCH1: track 0.00 -> 248.5 mm
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- added copper zone on B.Cu, net (none)
- added copper zone on F.Cu, net GND

Commit message: Resolved issues raised during DRC testing and compressed final files into zip
Parts:
- moved A1 1.22 mm to (308.1, 27.3)
Routing:
- net /ENC_B: track 279.5 -> 271.7 mm
- net /COL15: track 138.0 -> 143.8 mm
- net /COL14: track 124.8 -> 128.6 mm
- net /COL13: track 125.9 -> 129.6 mm
- net /COL8: track 223.3 -> 220.8 mm
- net /ROW0: track 350.1 -> 351.3 mm
- net /ENC_A: track 292.9 -> 294.1 mm
- net /ROW4: track 412.3 -> 413.5 mm
- net /ROW2: track 368.4 -> 369.6 mm
- net /ROW1: track 355.8 -> 357.0 mm
- net /ROW3: track 378.4 -> 379.6 mm
- net /COL12: track 151.1 -> 151.9 mm
- net /COL5: track 290.2 -> 289.5 mm
- net /COL0: track 440.7 -> 440.2 mm
- net /COL1: track 409.6 -> 409.1 mm
