File: keeb-kicad/keeb-kicad.kicad_pcb (KiCad board)
At the start: 2 copper layers, 329 x 135 mm, 147 parts, among them SW1 SW_Push, SW10 SW_Push, SW11 SW_Push, SW12 SW_Push, SW13 SW_Push, SW14 SW_Push, SW15 SW_Push, SW16 SW_Push, SW17 SW_Push, SW18 SW_Push, SW19 SW_Push, SW2 SW_Push, SW20 SW_Push, SW21 SW_Push, SW22 SW_Push, SW23 SW_Push, SW24 SW_Push, SW25 SW_Push, SW26 SW_Push, SW27 SW_Push, SW28 SW_Push, SW29 SW_Push, SW3 SW_Push, SW30 SW_Push, SW31 SW_Push, SW32 SW_Push, SW33 SW_Push, SW34 SW_Push, SW35 SW_Push, SW36 SW_Push, SW37 SW_Push, SW38 SW_Push, SW39 SW_Push, SW4 SW_Push, SW40 SW_Push, SW41 SW_Push, SW42 SW_Push, SW43 SW_Push, SW44 SW_Push, SW45 SW_Push, SW46 SW_Push, SW47 SW_Push, SW48 SW_Push, SW49 SW_Push, SW5 SW_Push, SW50 SW_Push, SW51 SW_Push, SW52 SW_Push, SW53 SW_Push, SW54 SW_Push, SW55 SW_Push, SW56 SW_Push, SW57 SW_Push, SW58 SW_Push, SW59 SW_Push, SW6 SW_Push, SW60 SW_Push, SW61 SW_Push, SW62 SW_Push, SW63 SW_Push, SW64 SW_Push, SW65 SW_Push, SW66 SW_Push, SW67 SW_Push, SW68 SW_Push, SW69 SW_Push, SW7 SW_Push, SW70 SW_Push, SW71 RotaryEncoder_Switch, SW8 SW_Push, SW9 SW_Push

Commit message: Finished up plate, added keycaps to render
Other:
- board size 329 x 135 mm -> 329 x 127.8 mm
Changed lines of the file:
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@@
 	(gr_rect
 		(start -19.05 19.05)
-		(end 309.9125 154.05)
+		(end 309.9125 146.81)
 		(stroke
 			(width 0.05)

Commit message: Added chamfers to PCB corners
Routing:
- net /COL0: track 440.2 -> 432.7 mm
Other:
- outline, holes or cut-outs redrawn
Changed lines of the file:
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@@
 		)
 	)
-	(gr_rect
-		(start -19.05 19.05)
-		(end 309.9125 146.81)
-		(stroke
-			(width 0.05)
-			(type default)
-		)
-		(fill no)
+	(gr_line
+		(start -19.0875 141.81)
+		(end -19.05 31.11)
+		(stroke
+			(width 0.05)
+			(type default)
+		)
+		(layer "Edge.Cuts")
+	)
+	(gr_line
+		(start -14.0875 146.81)
+		(end -19.0875 141.81)
+		(stroke
+			(width 0.05)
+			(type default)
+		)
+		(layer "Edge.Cuts")
+	)
+	(gr_line
+		(start -7.0875 19.11)
+		(end -19.05 31.11)
+		(stroke
+			(width 0.05)
+			(type default)
+		)
+		(layer "Edge.Cuts")
+	)
+	(gr_line
+		(start -7.0875 19.11)
+		(end 304.4477 19.05)
+		(stroke
+			(width 0.05)
+			(type default)
+		)
+		(layer "Edge.Cuts")
+	)
+	(gr_line
+		(start 302.2125 146.81)
+		(end -14.0875 146.81)
+		(stroke
+			(width 0.05)
+			(type default)
+		)
+		(layer "Edge.Cuts")
+	)
+	(gr_line
+		(start 304.5125 19.11)
+		(end 304.4477 19.05)
+		(stroke
+			(width 0.05)
+			(type default)
+		)
+		(layer "Edge.Cuts")
+	)
+	(gr_line
+		(start 309.9125 24.11)
+		(end 304.5125 19.11)
+		(stroke
+			(width 0.05)
+			(type default)
+		)
+		(layer "Edge.Cuts")
+	)
+	(gr_line
+		(start 309.9125 24.11)
+		(end 309.9125 139.11)
+		(stroke
+			(width 0.05)
+			(type default)
+		)
+		(layer "Edge.Cuts")
+	)
+	(gr_line
+		(start 309.9125 139.11)
+		(end 302.2125 146.81)
+		(stroke
+			(width 0.05)
+			(type default)
+		)
 		(layer "Edge.Cuts")
 	)
@@
 	)
 	(segment
+		(start -9.81 56.46)
+		(end -9.6875 56.3375)
+		(width 0.2)
+		(layer "B.Cu")
+		(net "/COL0")
+	)
+	(segment
 		(start -0.285 113.61)
 		(end -0.285 123.135)
@@
 	)
 	(segment
+		(start -5.0475 75.51)
+		(end -5.0475 92.17875)
+		(width 0.2)
+		(layer "B.Cu")
+		(net "/COL0")
+	)
+	(segment
+		(start -9.6875 56.3375)
+		(end -9.6875 35.21)
+		(width 0.2)
+		(layer "B.Cu")
+		(net "/COL0")
+	)
+	(segment
+		(start -2.66625 111.22875)
+		(end -0.285 113.61)
+		(width 0.2)
+		(layer "B.Cu")
+		(net "/COL0")
+	)
+	(segment
+		(start -9.81 56.46)
+		(end -9.81 70.7475)
+		(width 0.2)
+		(layer "B.Cu")
+		(net "/COL0")
+	)
+	(segment
+		(start -2.66625 94.56)
+		(end -2.66625 111.22875)
+		(width 0.2)
+		(layer "B.Cu")
+		(net "/COL0")
+	)
+	(segment
+		(start -0.285 123.135)
+		(end -9.81 132.66)
+		(width 0.2)
+		(layer "B.Cu")
+		(net "/COL0")
+	)
+	(segment
+		(start -5.0475 92.17875)
+		(end -2.66625 94.56)
+		(width 0.2)
+		(layer "B.Cu")
+		(net "/COL0")
+	)
+	(segment
 		(start 300.6125 19.81)
 		(end 308.1025 27.3)
@@
 	)
 	(segment
-		(start -9.81 22.5325)
-		(end -7.0875 19.81)
-		(width 0.2)
-		(layer "B.Cu")
-		(net "/COL0")
-	)
-	(segment
-		(start -5.0475 75.51)
-		(end -5.0475 92.17875)
-		(width 0.2)
-		(layer "B.Cu")
-		(net "/COL0")
-	)
-	(segment
-		(start -2.66625 111.22875)
-		(end -0.285 113.61)
-		(width 0.2)
-		(layer "B.Cu")
-		(net "/COL0")
-	)
-	(segment
-		(start -9.81 56.46)
-		(end -9.81 22.5325)
-		(width 0.2)
-		(layer "B.Cu")
-		(net "/COL0")
-	)
-	(segment
-		(start -9.81 56.46)
-		(end -9.81 70.7475)
-		(width 0.2)
-		(layer "B.Cu")
-		(net "/COL0")
-	)
-	(segment
-		(start -2.66625 94.56)
-		(end -2.66625 111.22875)
-		(width 0.2)
-		(layer "B.Cu")
-		(net "/COL0")
-	)
-	(segment
-		(start -0.285 123.135)
-		(end -9.81 132.66)
-		(width 0.2)
-		(layer "B.Cu")
-		(net "/COL0")
-	)
-	(segment
-		(start -5.0475 92.17875)
-		(end -2.66625 94.56)
-		(width 0.2)
-		(layer "B.Cu")
-		(net "/COL0")
-	)
-	(segment
 		(start -9.81 70.7475)
 		(end -5.0475 75.51)
@@
 	)
 	(segment
-		(start -7.0875 19.81)
+		(start 5.7125 19.81)
 		(end 300.6125 19.81)
 		(width 0.2)
 		(layer "B.Cu")
+		(net "/COL0")
+	)
+	(segment
+		(start -9.6875 35.21)
+		(end 5.7125 19.81)
+		(width 0.2)
+		(layer "B.Cu")
