File: keeb-kicad/keeb-kicad.kicad_pcb (KiCad board)
At the start: 2 copper layers, 329 x 127.8 mm, 147 parts, among them SW1 SW_Push, SW10 SW_Push, SW11 SW_Push, SW12 SW_Push, SW13 SW_Push, SW14 SW_Push, SW15 SW_Push, SW16 SW_Push, SW17 SW_Push, SW18 SW_Push, SW19 SW_Push, SW2 SW_Push, SW20 SW_Push, SW21 SW_Push, SW22 SW_Push, SW23 SW_Push, SW24 SW_Push, SW25 SW_Push, SW26 SW_Push, SW27 SW_Push, SW28 SW_Push, SW29 SW_Push, SW3 SW_Push, SW30 SW_Push, SW31 SW_Push, SW32 SW_Push, SW33 SW_Push, SW34 SW_Push, SW35 SW_Push, SW36 SW_Push, SW37 SW_Push, SW38 SW_Push, SW39 SW_Push, SW4 SW_Push, SW40 SW_Push, SW41 SW_Push, SW42 SW_Push, SW43 SW_Push, SW44 SW_Push, SW45 SW_Push, SW46 SW_Push, SW47 SW_Push, SW48 SW_Push, SW49 SW_Push, SW5 SW_Push, SW50 SW_Push, SW51 SW_Push, SW52 SW_Push, SW53 SW_Push, SW54 SW_Push, SW55 SW_Push, SW56 SW_Push, SW57 SW_Push, SW58 SW_Push, SW59 SW_Push, SW6 SW_Push, SW60 SW_Push, SW61 SW_Push, SW62 SW_Push, SW63 SW_Push, SW64 SW_Push, SW65 SW_Push, SW66 SW_Push, SW67 SW_Push, SW68 SW_Push, SW69 SW_Push, SW7 SW_Push, SW70 SW_Push, SW71 RotaryEncoder_Switch, SW8 SW_Push, SW9 SW_Push

Commit message: Completed layout, progress on new routing.
Parts:
- removed D69, D70: 1N4148, Diode_THT:D_DO-35_SOD27_P7.62mm_Horizontal
- removed SW70: SW_Push, PCM_marbastlib-mx:SW_MX_1u
- removed SW71: RotaryEncoder_Switch, Rotary_Encoder:RotaryEncoder_Alps_EC11E-Switch_Vertical_H20mm
- S1, S2: footprint PCM_marbastlib-mx:STAB_MX_P_2.75u -> PCM_marbastlib-mx:STAB_MX_P_2u
- S4: footprint PCM_marbastlib-mx:STAB_MX_P_3u -> PCM_marbastlib-mx:STAB_MX_P_2.25u
- SW69: value SW_Push -> RotaryEncoder_Switch; footprint PCM_marbastlib-mx:SW_MX_1u -> Rotary_Encoder:RotaryEncoder_Alps_EC11E-Switch_Vertical_H20mm
- moved D59 300.6 mm to (3.52, 138.0)
- moved SW59 300.6 mm to (-6.00, 135.2)
- moved SW31 291.1 mm to (3.52, 97.1)
- moved SW45 291.1 mm to (3.52, 116.2)
- moved D31 286.4 mm to (17.8, 100.0)
- moved D45 281.6 mm to (22.6, 119.0)
- moved SW64 71.4 mm to (191.6, 135.2)
- moved D64 71.4 mm to (201.2, 138.0)
- moved SW63 69.1 mm to (120.2, 135.2)
- moved D63 66.7 mm to (127.3, 138.0)
- moved D43 42.9 mm to (270.2, 99.9)
- moved SW69 38.3 mm to (301.5, 107.5)
- moved D56 38.1 mm to (251.2, 119.0)
- moved D65 33.3 mm to (232.1, 138.0)
- moved D66 33.3 mm to (251.2, 138.0)
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Connections:
- A1 pad 20: /COL15 -> unconnected-(A1-GPIO15-Pad20)
- A1 pad 25: /ROW0 -> /ROW4
- A1 pad 26: /ROW1 -> /ROW3
- A1 pad 29: /ROW3 -> /ROW1
- A1 pad 31: /ROW4 -> /ROW0
- D31 pad 1: /ROW1 -> /ROW2
- D45 pad 1: /ROW2 -> /ROW3
- D59 pad 1: /ROW3 -> /ROW4
- SW15 pad 1: /COL15 -> /COL14
- SW31 pad 1: /COL15 -> /COL0
- SW32 pad 1: /COL0 -> /COL1
- SW33 pad 1: /COL1 -> /COL2
- SW34 pad 1: /COL2 -> /COL3
- SW35 pad 1: /COL3 -> /COL4
- SW36 pad 1: /COL4 -> /COL5
- SW37 pad 1: /COL5 -> /COL6
- SW38 pad 1: /COL6 -> /COL7
- SW39 pad 1: /COL7 -> /COL8
- SW40 pad 1: /COL8 -> /COL9
- SW41 pad 1: /COL9 -> /COL10
- SW42 pad 1: /COL10 -> /COL11
- SW43 pad 1: /COL11 -> /COL13
- SW44 pad 1: /COL13 -> /COL14
- SW45 pad 1: /COL15 -> /COL0
- SW46 pad 1: /COL0 -> /COL1
- SW47 pad 1: /COL1 -> /COL2
- SW48 pad 1: /COL2 -> /COL3
- SW49 pad 1: /COL3 -> /COL4
- SW50 pad 1: /COL4 -> /COL5
- SW51 pad 1: /COL5 -> /COL6
- SW52 pad 1: /COL6 -> /COL7
- SW53 pad 1: /COL7 -> /COL8
- SW54 pad 1: /COL8 -> /COL9
- SW55 pad 1: /COL9 -> /COL10
- SW56 pad 1: /COL10 -> /COL11
- SW57 pad 1: /COL12 -> /COL13
- SW59 pad 1: /COL15 -> /COL0
- SW60 pad 1: /COL0 -> /COL1
- SW61 pad 1: /COL1 -> /COL2
- SW62 pad 1: /COL2 -> /COL3
- SW63 pad 1: /COL3 -> /COL6
- SW64 pad 1: /COL6 -> /COL10
- SW65 pad 1: /COL10 -> /COL11
- SW66 pad 1: /COL11 -> /COL12
- SW67 pad 1: /COL12 -> /COL13
- SW68 pad 1: /COL13 -> /COL14
Routing:
- net /ENC_A: track 294.1 -> 56.4 mm
- net /SWITCH1: track 248.0 -> 18.0 mm
- net /ENC_B: track 271.7 -> 42.2 mm
- net /ROW0: track 351.3 -> 514.0 mm
- net /COL15: track 143.8 -> 0.00 mm
- net /COL14: track 128.6 -> 52.0 mm
- net /ROW2: track 369.6 -> 309.6 mm
- net /ROW3: track 379.6 -> 319.8 mm
- net /ROW4: track 413.5 -> 355.0 mm
- net /COL10: track 199.4 -> 143.7 mm
- net /COL11: track 173.6 -> 121.3 mm
- net /COL13: track 129.6 -> 77.4 mm
- net /ROW1: track 357.0 -> 307.0 mm
- net /COL12: track 151.9 -> 102.6 mm
- net /COL9: track 198.9 -> 161.2 mm
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Other:
- board size 329 x 127.8 mm -> 342.5 x 127.5 mm

Commit message: Finished and exported PCB
Parts:
- moved D63 2.45 mm to (129.8, 138.1)
Routing:
- net /COL11: track 121.3 -> 193.0 mm
- net /COL10: track 143.7 -> 209.8 mm
- net /COL13: track 77.4 -> 142.4 mm
- net /COL12: track 102.6 -> 163.7 mm
- net /COL14: track 52.0 -> 109.2 mm
- net /COL9: track 161.2 -> 203.3 mm
- net GND: track 0.00 -> 26.4 mm
- net Net-(D43-A): track 0.00 -> 19.7 mm
- net Net-(D56-A): track 0.00 -> 17.7 mm
- net Net-(D14-A): track 0.00 -> 17.4 mm
- net Net-(D45-A): track 0.00 -> 17.4 mm
- net /ENC_A: track 56.4 -> 71.8 mm
- net Net-(D16-A): track 0.00 -> 12.0 mm
- net Net-(D31-A): track 0.00 -> 11.9 mm
- net Net-(D65-A): track 0.00 -> 11.9 mm
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- added copper zone on B.Cu, net GND
- removed copper zone on B.Cu, net (none)
Other:
- board size 342.5 x 127.5 mm -> 342.5 x 101.5 mm
